File: hardware/DAS.kicad_pcb (KiCad board)
At the start: 2 copper layers, 150 x 70 mm, 173 parts, among them P1 CONN_01X04, P10 CONN_01X02, P11 CONN_01X04, P12 CONN_01X02, P13 CONN_01X03, P2 CONN_02X03, P3 CONN_01X03, P4 CONN_01X02, P5 CONN_01X02, P6 CONN_01X02, P7 CONN_01X02, P8 CONN_01X02, P9 CONN_01X02, U1 7805, U10 ASSR_45_1228_45_002, U11 ASSR_45_1228_45_002, U12 ASSR_45_1228_45_002, U13 MAX13053ESA+, U14 ASSR_45_1228_45_002, U15 MC9S08DZ_LC, U16 G3VM-61ER, U17 LP5907_DBV_5, U18 LP5907_DBV_5, U19 SN74HC138_PW_16, U2 LP5907_DBV_5, U20 SST25VF512A-33-4, U21 SN74LV1T125DBVR, U22 G5V_45_1_32_12DC, U23 DS18B20, U3 ADUM5401ARWZ, U4 AD7792BRUZ, U5 SN74LV1T125DBVR, U6 ASSR_45_1228_45_002, U7 ASSR_45_1228_45_002, U8 ASSR_45_1228_45_002, U9 ASSR_45_1228_45_002, Y1 8MHz

Commit message: Try fix issues found out during prototyping.   Misused LDO supplying VDDA removed.   Wrong pin assignment to DC-DC module corrected.   Footprint of SPI Flash tweaked to allow wider selection of parts.   A pull-up resistor and a current limit resistor added to Chain block.   Footprint SOD-323 changed to KiCad's one.   The main power capacitor has been splitted to two.
Parts:
- removed C68: 0.1u, Capacitors_SMD:C_0805
- removed P13: CONN_01X03, Pin_Headers:Pin_Header_Straight_1x03
- removed R47: 6k8, Resistors_SMD:R_0805
- removed U17: LP5907_DBV_5, footprints:LP5907_DBV_5
- removed U22: G5V_45_1_32_12DC, footprints:G5V-1_12DC
- removed U23: DS18B20, footprints:ds18s20
- added C0: 470u, Capacitors_SMD:c_elec_10x10.5, F.Cu at (102.8, 120.6)
- C1: value 1000u -> 470u; footprint footprints:c_elec_16x16.5 -> Capacitors_SMD:c_elec_10x10.5
- D18, D3, D4: footprint footprints:SOD-323 -> Diodes_SMD:SOD-323
- R38: value 4k7 -> 0
- R46: value 4k7 -> 0; moved to F.Cu
- R48, R49, R50: value 2k -> 2k2
- U20: footprint footprints:SST25VF512A-33-4 -> Housings_SOIC:SOIJ-8_5.3x5.3mm_Pitch1.27mm
- moved R46 130.0 mm to (221.8, 114.9), turned to 270 degrees
- moved R45 23.7 mm to (208.5, 120.9), turned to 0 degrees
- moved D1 14.8 mm to (94.7, 123.3), turned to 90 degrees
- moved D2 9.91 mm to (91.0, 120.0), turned to 90 degrees
- moved C8 7.83 mm to (94.7, 118.9), turned to 90 degrees
- moved R38 4.46 mm to (160.4, 111.0), turned to 0 degrees
- moved C1 3.67 mm to (114.2, 120.6), turned to 270 degrees
- moved C3 2.80 mm to (134.6, 119.7), turned to 270 degrees
- moved C4 2.80 mm to (136.7, 119.7), turned to 270 degrees
- moved C5 2.80 mm to (138.7, 119.7), turned to 270 degrees
- moved C2 2.72 mm to (122.7, 122.1), turned to 90 degrees
- moved R48 0.70 mm to (113.2, 71.7)
- moved R40 0.30 mm to (125.8, 69.0)
- moved R44 0.28 mm to (113.0, 69.1)
- moved U1 0.05 mm to (131.3, 118.4)
Connections:
- net CANH renamed CAN+
- net CANL renamed CAN-
- C1 pad 1: Net-(C1-Pad1) -> Net-(C0-Pad1)
- C2 pad 1: Net-(C1-Pad1) -> Net-(C0-Pad1)
- C8 pad 1: +12V -> VPP
- D1 pad 1: Net-(C1-Pad1) -> Net-(C0-Pad1)
- D1 pad 2: +12V -> VPP
- D2 pad 1: +12V -> VPP
- R38 pad 2: Net-(R38-Pad2) -> VDDA
- R46 pad 1: GNDD -> Net-(P11-Pad2)
- R46 pad 2: GPIO0 -> Net-(R46-Pad2)
- U1 pad 1: Net-(C1-Pad1) -> +5VD
- U1 pad 3: +5VD -> Net-(C0-Pad1)
- U16 pad 6: Net-(P11-Pad2) -> Net-(R46-Pad2)
Routing:
- net GPIO0: track 96.1 -> 2.27 mm
- net GNDD: track 1260.4 -> 1216.9 mm
- net Net-(C0-Pad1): track 0.00 -> 37.6 mm
- net Net-(C1-Pad1): track 35.3 -> 0.00 mm
- net /PWM: track 16.4 -> 0.00 mm
- net GPIO1: track 51.1 -> 40.6 mm, vias 3 -> 2
- net +12V: track 8.79 -> 0.00 mm
- net +5VD: track 795.5 -> 788.3 mm
- net /EN: track 6.66 -> 0.00 mm
- net Net-(P11-Pad2): track 5.16 -> 10.7 mm
- net VPP: track 149.2 -> 152.1 mm
- net Net-(R46-Pad2): track 0.00 -> 2.54 mm
- net Net-(R38-Pad2): track 1.58 -> 0.00 mm
- net Net-(R43-Pad2): track 10.5 -> 9.36 mm
- net Net-(R41-Pad2): track 7.24 -> 6.13 mm
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Other:
- board text added: "PCB V1R2"
- board text removed: "PCB V1R1"
