File: hardware/DAS.sch (KiCad schematic (older format))
At the start: 173 parts, among them P1 CONN_01X04, P10 CONN_01X02, P11 CONN_01X04, P12 CONN_01X02, P13 CONN_01X03, P2 CONN_02X03, P3 CONN_01X03, P4 CONN_01X02, P5 CONN_01X02, P6 CONN_01X02, P7 CONN_01X02, P8 CONN_01X02, P9 CONN_01X02, U1 7805, U10 ASSR_45_1228_45_002, U11 ASSR_45_1228_45_002, U12 ASSR_45_1228_45_002, U13 MAX13053ESA+, U14 ASSR_45_1228_45_002, U15 MC9S08DZ_LC, U16 G3VM-61ER, U17 LP5907_DBV_5, U18 LP5907_DBV_5, U19 SN74HC138_PW_16, U2 LP5907_DBV_5, U20 SST25VF512A-33-4, U21 SN74LV1T125DBVR, U22 G5V_45_1_32_12DC, U23 DS18B20, U3 ADUM5401ARWZ, U4 AD7792BRUZ, U5 SN74LV1T125DBVR, U6 ASSR_45_1228_45_002, U7 ASSR_45_1228_45_002, U8 ASSR_45_1228_45_002, U9 ASSR_45_1228_45_002, Y1 8MHz

Commit message: Try fix issues found out during prototyping.   Misused LDO supplying VDDA removed.   Wrong pin assignment to DC-DC module corrected.   Footprint of SPI Flash tweaked to allow wider selection of parts.   A pull-up resistor and a current limit resistor added to Chain block.   Footprint SOD-323 changed to KiCad's one.   The main power capacitor has been splitted to two.
Parts:
- removed C68: 0.1u, Capacitors_SMD:C_0805, symbol C
- removed P13: CONN_01X03, Pin_Headers:Pin_Header_Straight_1x03, symbol CONN_01X03
- removed R47: 6k8, Resistors_SMD:R_0805, symbol R
- removed U17: LP5907_DBV_5, footprints:LP5907_DBV_5, symbol LP5907_DBV_5
- removed U22: G5V_45_1_32_12DC, footprints:G5V-1_12DC, symbol G5V_45_1_32_12DC
- removed U23: DS18B20, footprints:ds18s20, symbol DS18S20_43_
- added C0: 470u, Capacitors_SMD:c_elec_10x10.5, symbol CP
- C1: value 1000u -> 470u; footprint footprints:c_elec_16x16.5 -> Capacitors_SMD:c_elec_10x10.5
- R38, R46: value 4k7 -> 0
Connections:
- net +12V is gone; now on net VPP: C8.1, D1.2 (A), D2.1
- net GNDD: now also C0.2; no longer R46.1
- net GPIO0: no longer R46.2
- net VDDA: now also R38.2
- net at C1.1, C2.1, D1.1 (K)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: now also C0.1
- net at P11.2 (P2): now also R46.1; no longer U16.6 (INOUT2)
- net CANH renamed CAN+
- net CANL renamed CAN-
- new net: R46.2, U16.6 (INOUT2)
- no-connect marks 13 -> 12
Other:
- note added: "940uF > 50ms*100mA/(11V-5V)"
- note removed: "1000uF > 50ms*100mA/(11V-5V)"
- note removed: "For PATAC"
- moved on the sheet: C54, C55, C61, C8, D1, D2, R38, R45
